File: boards/test_hard/adc.kicad_sch (KiCad schematic)
At the start: 26 parts, among them IC1 ADS114S08BIPBS, J1 Sensor 1, J2 Sensor 2, J3 ACOM

Commit message: 1Ohm res and stencil
Parts:
- added R17, R18: 1, Resistor_SMD:R_0603_1608Metric_Pad0.98x0.95mm_HandSolder, symbol Device:R
Connections:
- net D1N: now also R17.1
- net D1P: now also R17.2
- net D2N: now also R18.1
- net D2P: now also R18.2
Other:
- moved on the sheet: J1, J2

Commit message: Aktueller Stand
Signed-off-by: Philipp Macher <philipp-macher@web.de>
Other:
- moved on the sheet: J1, J2, J3, JP1, R17, R18, R6, R7
